Commit message: Update robots URDF

File: ur3e_dual_description/urdf/dual_ur3e_flat.urdf.xacro (robot description, xacro)
@@ -2,12 +2,12 @@
 <robot xmlns:xacro="http://ros.org/wiki/xacro"
        name="ur3e" >
+  <!--  Author: Cristian Beltran -->
   <!-- Arguments -->
   <xacro:arg name="grasp_plugin" default="false" />
-  <xacro:arg name="transmission_hw_interface" default="hardware_interface/PositionJointInterface"/>
-  <xacro:arg name="kinematics_config" default="$(find ur_e_description)/config/ur3e_default.yaml"/>
+  <xacro:arg name="use_effort_interface" default="false" />
   <!-- common stuff -->
-  <xacro:include filename="$(find ur_e_description)/urdf/common.gazebo.xacro" />
+  <xacro:include filename="$(find ur3_description)/urdf/common.gazebo.xacro" />
   <!-- ur3e -->
-  <xacro:include filename="$(find ur_e_description)/urdf/ur3e.urdf.xacro" />
+  <xacro:include filename="$(find ur3_description)/urdf/ur3e/ur3e.urdf.xacro" />
   <!-- arm -->
   <xacro:ur3e_robot prefix="leftarm_" joint_limited="true"
@@ -18,6 +18,4 @@
     wrist_2_lower_limit="${-pi}" wrist_2_upper_limit="${pi}"
     wrist_3_lower_limit="${-2*pi}" wrist_3_upper_limit="${2*pi}"
-    transmission_hw_interface="$(arg transmission_hw_interface)"
-    kinematics_file="${load_yaml('$(arg kinematics_config)')}"
   />
   <xacro:ur3e_robot prefix="rightarm_" joint_limited="true"
@@ -28,6 +26,4 @@
     wrist_2_lower_limit="${-pi}" wrist_2_upper_limit="${pi}"
     wrist_3_lower_limit="${-2*pi}" wrist_3_upper_limit="${2*pi}"
-    transmission_hw_interface="$(arg transmission_hw_interface)"
-    kinematics_file="${load_yaml('$(arg kinematics_config)')}"
   />
   <!-- Include workspace -->
@@ -49,3 +45,7 @@
     <origin xyz="0.5 -0.45 1.0" rpy="0 0 0" />
   </joint>
+  <!-- spawn and attach dual robotiq 85 grippers (two different macros are used because different tool frames are defined inside) -->
+  <xacro:include filename="$(find ur3e_dual_description)/urdf/robotiq_hande_gripper_manual_exchanger.urdf.xacro" />
+  <xacro:robotiq_hande_gripper_adapter prefix="leftarm_" parent = "leftarm_ee_link" />
+  <xacro:robotiq_hande_gripper_adapter prefix="rightarm_" parent = "rightarm_ee_link" />
 </robot>

File: ur3e_dual_description/urdf/kosmek_manual_exchanger.urdf.xacro (robot description, xacro)
@@ -1,7 +1,5 @@
 <?xml version="1.0"?>
 <robot xmlns:xacro="http://ros.org/wiki/xacro">
-  <!--
-  Author: Cristian Beltran
--->
+  <!--  Author: Cristian Beltran -->
   <xacro:macro name="kosmek_exchanger" params="prefix parent *origin">
     <joint name="${prefix}kosmek_base_joint" type="fixed">

File: ur3e_dual_description/urdf/robotiq_hande_gripper.urdf.xacro (robot description, xacro)
@@ -3,15 +3,10 @@
 <!-- This macro adds a convenient TF frame at the tip of the closed gripper. -->
 <!-- The position of the TF frame has not been measured at all and needs to be calibrated. -->
-<robot name="robotiq_hande_gripper_adapter_manual_exchanger"
+<robot name="robotiq_hande_gripper_adapter"
     xmlns:xacro="http://www.ros.org/wiki/xacro">
     <!-- This seems too long when measuring the sensor,
        but works out when calibrating the tip_link to the world. -->
-    <xacro:macro name="robotiq_hande_gripper_adapter_manual_exchanger" params="prefix parent ft_prefix">
+    <xacro:macro name="robotiq_hande_gripper_adapter" params="prefix parent ft_prefix">
         <xacro:include filename="$(find robotiq_description)/urdf/robotiq_hande_gripper.urdf.xacro" />
-        <xacro:include filename="$(find ur3e_dual_description)/urdf/kosmek_manual_exchanger.urdf.xacro" />
-        <!-- tool exchanger -->
-        <xacro:kosmek_exchanger prefix="${prefix}" parent="${prefix}tool0">
-            <origin xyz="0 0.0 0.0025" rpy="0 ${pi/2.0} 0" />
-        </xacro:kosmek_exchanger>
         <link name="${prefix}robotiq_coupler">
             <visual>
@@ -33,6 +28,6 @@
         </link>
         <joint name="${prefix}robotiq_coupler_joint" type="fixed">
-            <origin xyz="-0.0405 0.0 0" rpy="0 ${-pi/2.0} 0" />
-            <parent link="${prefix}kosmek_exchanger_base_link"/>
+            <origin xyz="0 0 0.004" rpy="0 0 ${-pi/2.0}" />
+            <parent link="${prefix}tool0"/>
             <child link="${prefix}robotiq_coupler"/>
         </joint>
@@ -43,13 +38,13 @@
         </gazebo>
         <!-- Add additional links for us to plan with. Oriented like the UR frame. -->
-        <link name="${prefix}gripper_tip_link" />
+        <link name="${prefix}robotiq_hande_tip_link_joint" />
         <joint name="${prefix}manipulator_dummy_joint" type="fixed">
             <parent link="${prefix}robotiq_coupler"/>
-            <child link="${prefix}gripper_tip_link"/>
+            <child link="${prefix}robotiq_hande_tip_link_joint"/>
             <origin xyz="0 0 0.1441" rpy="0 0 0" />
         </joint>
         <!-- Attach the robotiq hand-e gripper -->
-        <xacro:robotiq_hande_gripper prefix="${prefix}" parent="${prefix}robotiq_coupler">
-            <origin xyz="0 0 0.004" rpy="0 0 0"/>
+        <xacro:robotiq_hande_gripper prefix="${prefix}" parent="${parent}">
+            <origin xyz="0 0 0.004" rpy="${pi/2.0} 0 ${pi/2}"/>
         </xacro:robotiq_hande_gripper>
         <!-- Gazebo FT sensor plugin -->
@@ -62,5 +57,5 @@
                 <topicName>${ft_prefix}/wrench</topicName>
                 <gaussianNoise>0.0</gaussianNoise>
-                <jointName>${prefix}wrist_3_joint</jointName>
+                <jointName>${prefix}wrist_3_link-tool0_fixed_joint</jointName>
             </plugin>
         </gazebo>

File: ur3e_dual_description/urdf/single_ur3e.urdf.xacro (robot description, xacro)
@@ -11,5 +11,5 @@
   <xacro:include filename="$(find ur3_description)/urdf/ur3e/ur3e.urdf.xacro" />
   <!-- arm -->
-  <xacro:ur3e_robot prefix="leftarm_" joint_limited="true"
+  <xacro:ur3e_robot prefix="" joint_limited="true"
     shoulder_pan_lower_limit="${0}" shoulder_pan_upper_limit="${2*pi}"
     shoulder_lift_lower_limit="${-pi}" shoulder_lift_upper_limit="${pi}"
@@ -18,12 +18,4 @@
     wrist_2_lower_limit="${-pi}" wrist_2_upper_limit="${pi}"
     wrist_3_lower_limit="${-2*pi}" wrist_3_upper_limit="${2*pi}"
-  />
-  <xacro:ur3e_robot prefix="rightarm_" joint_limited="true"
-    shoulder_pan_lower_limit="${0}" shoulder_pan_upper_limit="${2*pi}"
-    shoulder_lift_lower_limit="${-pi}" shoulder_lift_upper_limit="${pi}"
-    elbow_joint_lower_limit="${-pi}" elbow_joint_upper_limit="${pi}"
-    wrist_1_lower_limit="${-pi}" wrist_1_upper_limit="${pi}"
-    wrist_2_lower_limit="${-pi}" wrist_2_upper_limit="${pi}"
-    wrist_3_lower_limit="${-10*pi}" wrist_3_upper_limit="${10*pi}"
   />
   <!-- Include workspace -->
@@ -35,18 +27,12 @@
   </joint>
   <link name="world" />
-  <joint name="world_leftarm_joint" type="fixed">
+  <joint name="world_joint" type="fixed">
     <parent link="world" />
-    <child link="leftarm_base_link" />
+    <child link="base_link" />
     <origin xyz="0.365 0.345 1.330" rpy="1.5707 0.0 1.5707" />
-  </joint>
-  <joint name="world_rightarm_joint" type="fixed">
-    <parent link="world" />
-    <child link = "rightarm_base_link" />
-    <origin xyz="0.365 -0.345 1.330" rpy="1.5707 0.0 1.5707" />
   </joint>
   <!-- spawn and attach dual robotiq 85 grippers (two different macros are used because different tool frames are defined inside) -->
   <xacro:include filename="$(find ur3e_dual_description)/urdf/robotiq_hande_gripper_manual_exchanger.urdf.xacro" />
   <!-- <xacro:include filename="$(find ur3e_dual_description)/urdf/robotiq_hande_gripper.urdf.xacro" /> -->
-  <xacro:robotiq_hande_gripper_adapter_manual_exchanger prefix="leftarm_" parent = "leftarm_ee_link" ft_prefix="leftarm"/>
-  <xacro:robotiq_hande_gripper_adapter_manual_exchanger prefix="rightarm_" parent = "rightarm_ee_link" ft_prefix="rightarm"/>
+  <xacro:robotiq_hande_gripper_adapter_manual_exchanger prefix="" parent = "ee_link" ft_prefix=""/>
 </robot>

File: ur3e_dual_description/urdf/ur3e_dual_flat_workspace.urdf.xacro (robot description, xacro)
@@ -1,125 +1,125 @@
 <?xml version="1.0"?>
+  <!--  Author: Cristian Beltran -->
 <!-- This macro adds a convenient TF frame at the tip of the closed gripper. -->
 <!-- The position of the TF frame has not been measured at all and needs to be calibrated. -->
-<robot name="ur3e_dual_workspace" xmlns:xacro="http://www.ros.org/wiki/xacro">
-    <link name="workspace_table">
-            <visual>
-            <geometry>
-                <mesh filename="package://ur3e_dual_description/meshes/ur3e_table.stl" />
-            </geometry>
-            <material name="dark_gray">
-            <color rgba="${100/255} ${100/255} ${100/255} 1.0"/>
-            </material>
-            </visual>
-            <collision>
-            <geometry>
-                <mesh filename="package://ur3e_dual_description/meshes/ur3e_table.stl" />
-            </geometry>
-            </collision>
-            <inertial>
-            <origin xyz="0.401616 -0.000430 0.525458" rpy="0 0 0" />
-            <mass value="10.0" />
-            <inertia ixx="0.054454" ixy="-0.000007" ixz="0.005301"
-                    iyy="0.034120" iyz="0.000009" izz="0.046806"/>
-            </inertial>
-    </link>
-    <link name="workspace_tool_holder">
-        <visual>
-        <geometry>
-            <mesh filename="package://ur3e_dual_description/meshes/simple_tool_support.stl" />
-        </geometry>
-        <material name="transparent">
-          <color rgba="${150/255} ${150/255} ${150/255} 0.7"/>
-        </material>
-        </visual>
-        <collision>
-        <geometry>
-            <mesh filename="package://ur3e_dual_description/meshes/simple_tool_support.stl" />
-        </geometry>
-        </collision>
-        <inertial>
-        <origin xyz="0.401616 -0.000430 0.525458" rpy="0 0 0" />
-        <mass value="10.0" />
-        <inertia ixx="0.054454" ixy="-0.000007" ixz="0.005301"
-                iyy="0.034120" iyz="0.000009" izz="0.046806"/>
-        </inertial>
-    </link>
-    <link name="rightarm_support">
-      <visual>
-        <origin xyz="0.0 0.0 0.11" rpy="0 0 0"/>
-        <geometry>
-          <box size="0.1 0.1 0.22"/>
-        </geometry>
-        <material name="transparent">
-          <color rgba="${150/255} ${150/255} ${150/255} 0.7"/>
-        </material>
-      </visual>
-      <collision>
-        <origin xyz="0.0 0.0 0.11" rpy="0 0 0"/>
-        <geometry>
-          <box size="0.1 0.1 0.22"/>
-        </geometry>
-      </collision>
-      <inertial>
-        <mass value="2.0" />
-        <origin xyz="0.0 0.0 0.0" />
-        <inertia ixx = "1.0" ixy = "0.000000" ixz = "0.000000"
+<robot name="ur3e_dual_workspace"
+  xmlns:xacro="http://www.ros.org/wiki/xacro">
+  <link name="workspace_table">
+    <visual>
+      <geometry>
+        <mesh filename="package://ur3e_dual_description/meshes/ur3e_table.stl" />
+      </geometry>
+      <material name="dark_gray">
+        <color rgba="${100/255} ${100/255} ${100/255} 1.0"/>
+      </material>
+    </visual>
+    <collision>
+      <geometry>
+        <mesh filename="package://ur3e_dual_description/meshes/ur3e_table.stl" />
+      </geometry>
+    </collision>
+    <inertial>
+      <origin xyz="0.401616 -0.000430 0.525458" rpy="0 0 0" />
+      <mass value="10.0" />
+      <inertia ixx="0.054454" ixy="-0.000007" ixz="0.005301" iyy="0.034120" iyz="0.000009" izz="0.046806"/>
+    </inertial>
+  </link>
+  <link name="workspace_tool_holder">
+    <visual>
+      <geometry>
+        <mesh filename="package://ur3e_dual_description/meshes/simple_tool_support.stl" />
+      </geometry>
+      <material name="transparent">
+        <color rgba="${150/255} ${150/255} ${150/255} 0.7"/>
+      </material>
+    </visual>
+    <collision>
+      <geometry>
+        <mesh filename="package://ur3e_dual_description/meshes/simple_tool_support.stl" />
+      </geometry>
+    </collision>
+    <inertial>
+      <origin xyz="0.401616 -0.000430 0.525458" rpy="0 0 0" />
+      <mass value="10.0" />
+      <inertia ixx="0.054454" ixy="-0.000007" ixz="0.005301" iyy="0.034120" iyz="0.000009" izz="0.046806"/>
+    </inertial>
+  </link>
+  <link name="rightarm_support">
+    <visual>
+      <origin xyz="0.0 0.0 0.11" rpy="0 0 0"/>
+      <geometry>
+        <box size="0.1 0.1 0.22"/>
+      </geometry>
+      <material name="transparent">
+        <color rgba="${150/255} ${150/255} ${150/255} 0.7"/>
+      </material>
+    </visual>
+    <collision>
+      <origin xyz="0.0 0.0 0.11" rpy="0 0 0"/>
+      <geometry>
+        <box size="0.1 0.1 0.22"/>
+      </geometry>
+    </collision>
+    <inertial>
+      <mass value="2.0" />
+      <origin xyz="0.0 0.0 0.0" />
+      <inertia ixx = "1.0" ixy = "0.000000" ixz = "0.000000"
              iyx = "0.000000" iyy = "1.0" iyz = "0.000000"
              izx = "0.000000" izy = "0.000000" izz = "1.0" />
-      </inertial>
-    </link>
-    <link name="leftarm_support">
-      <visual>
-        <origin xyz="0.0 0.0 0.11" rpy="0 0 0"/>
-        <geometry>
-          <box size="0.1 0.1 0.22"/>
-        </geometry>
-        <material name="transparent">
-          <color rgba="${150/255} ${150/255} ${150/255} 0.7"/>
-        </material>
-      </visual>
-      <collision>
-        <origin xyz="0.0 0.0 0.11" rpy="0 0 0"/>
-        <geometry>
-          <box size="0.1 0.1 0.22"/>
-        </geometry>
-      </collision>
-      <inertial>
-        <mass value="2.0" />
-        <origin xyz="0.0 0.0 0.0" />
-        <inertia ixx = "1.0" ixy = "0.000000" ixz = "0.000000"
+    </inertial>
+  </link>
+  <link name="leftarm_support">
+    <visual>
+      <origin xyz="0.0 0.0 0.11" rpy="0 0 0"/>
+      <geometry>
+        <box size="0.1 0.1 0.22"/>
+      </geometry>
+      <material name="transparent">
+        <color rgba="${150/255} ${150/255} ${150/255} 0.7"/>
+      </material>
+    </visual>
+    <collision>
+      <origin xyz="0.0 0.0 0.11" rpy="0 0 0"/>
+      <geometry>
+        <box size="0.1 0.1 0.22"/>
+      </geometry>
+    </collision>
+    <inertial>
+      <mass value="2.0" />
+      <origin xyz="0.0 0.0 0.0" />
+      <inertia ixx = "1.0" ixy = "0.000000" ixz = "0.000000"
              iyx = "0.000000" iyy = "1.0" iyz = "0.000000"
              izx = "0.000000" izy = "0.000000" izz = "1.0" />
-      </inertial>
-    </link>
-    <joint name="workspace_table_rightarm_support_joint" type="fixed">
-        <parent link="workspace_table" />
-        <child link="rightarm_support" />
-        <origin xyz="0.50 -0.45 0.78" rpy="0.0 0.0 0.0" />
-    </joint>
-    <joint name="workspace_table_leftarm_support_joint" type="fixed">
-        <parent link="workspace_table" />
-        <child link="leftarm_support" />
-        <origin xyz="0.50 0.45 0.78" rpy="0.0 0.0 0.0" />
-    </joint>
-    <joint name="workspace_table_tool_holder_joint" type="fixed">
-        <parent link="workspace_table" />
-        <child link="workspace_tool_holder" />
-        <origin xyz="0.96 0.20 0.75" rpy="1.5707 0.0 3.1415" />
-    </joint>
-    <gazebo reference="workspace_body">
-        <mu1>0.9</mu1>
-        <mu2>0.9</mu2>
-        <material>Gazebo/BlueTransparent</material>
-    </gazebo>
-        <gazebo reference="workspace_table">
-        <mu1>0.9</mu1>
-        <mu2>0.9</mu2>
-        <material>Gazebo/DarkGrey</material>
-    </gazebo>
-        <gazebo reference="workspace_tool_holder">
-        <mu1>0.9</mu1>
-        <mu2>0.9</mu2>
-        <material>Gazebo/GreyTransparent</material>
-    </gazebo>
+    </inertial>
+  </link>
+  <joint name="workspace_table_rightarm_support_joint" type="fixed">
+    <parent link="workspace_table" />
+    <child link="rightarm_support" />
+    <origin xyz="0.50 -0.45 0.78" rpy="0.0 0.0 0.0" />
+  </joint>
+  <joint name="workspace_table_leftarm_support_joint" type="fixed">
+    <parent link="workspace_table" />
+    <child link="leftarm_support" />
+    <origin xyz="0.50 0.45 0.78" rpy="0.0 0.0 0.0" />
+  </joint>
+  <joint name="workspace_table_tool_holder_joint" type="fixed">
+    <parent link="workspace_table" />
+    <child link="workspace_tool_holder" />
+    <origin xyz="0.96 0.20 0.75" rpy="1.5707 0.0 3.1415" />
+  </joint>
+  <gazebo reference="workspace_body">
+    <mu1>0.9</mu1>
+    <mu2>0.9</mu2>
+    <material>Gazebo/GreyTransparent</material>
+  </gazebo>
+  <gazebo reference="workspace_table">
+    <mu1>0.9</mu1>
+    <mu2>0.9</mu2>
+    <material>Gazebo/DarkGrey</material>
+  </gazebo>
+  <gazebo reference="workspace_tool_holder">
+    <mu1>0.9</mu1>
+    <mu2>0.9</mu2>
+    <material>Gazebo/GreyTransparent</material>
+  </gazebo>
 </robot>
